Commit message: Add Depth Camera

File: echo_bot_pkg/description/depth_camera.xacro (robot description, xacro)
@@ -4,5 +4,5 @@
         <parent link="chassis"/>
         <child link="camera_link"/>
-        <origin xyz="0.505 0 0.1" rpy="0 0.0 0"/>
+        <origin xyz="0.505 0 0.1" rpy="0 0 0"/>
     </joint>
     <link name="camera_link">
@@ -22,5 +22,5 @@
     <gazebo reference="camera_link">
         <material>Gazebo/White</material>
-        <sensor name="camera" type="camera">
+        <sensor name="camera" type="depth">
             <pose> 0 0 0 0 0 0 </pose>
             <visualize>true</visualize>
@@ -29,5 +29,5 @@
                 <horizontal_fov>1.089</horizontal_fov>
                 <image>
-                    <format>R8G8B8</format>
+                    <format>B8G8R8</format>
                     <width>640</width>
                     <height>480</height>
@@ -40,4 +40,6 @@
             <plugin name="camera_controller" filename="libgazebo_ros_camera.so">
                 <frame_name>camera_optical_link</frame_name>
+                <min_depth>0.1</min_depth>
+                <max_depth>100</max_depth>
             </plugin>
         </sensor>

File: echo_bot_pkg/description/robot.urdf.xacro (robot description, xacro)
@@ -4,6 +4,8 @@
     <xacro:include filename="gazebo_control.xacro" />
     <xacro:include filename="lidar.xacro" />
-    <xacro:include filename="camera.xacro" />
+    <!-- To use camera, comment out depth camera and use the camera xacro tag. -->
+    <!-- <xacro:include filename="camera.xacro" /> -->
+    <xacro:include filename="depth_camera.xacro" />
     <!-- <xacro:include filename="ros2_control.xacro" />
-     <xacro:include filename="depth_camera.xacro" />  -->
+       -->
 </robot>
