Commit message: ROS2 Control

File: echo_bot_pkg/description/robot.urdf.xacro (robot description, xacro)
@@ -2,10 +2,10 @@
 <robot xmlns:xacro="http://www.ros.org/wiki/xacro"  name="robot">
     <xacro:include filename="robot_base.xacro" />
-    <xacro:include filename="gazebo_control.xacro" />
     <xacro:include filename="lidar.xacro" />
     <!-- To use camera, comment out depth camera and use the camera xacro tag. -->
     <!-- <xacro:include filename="camera.xacro" /> -->
     <xacro:include filename="depth_camera.xacro" />
-    <!-- <xacro:include filename="ros2_control.xacro" />
-       -->
+    <!-- Commenting Gazebo Control so that ros2_control can be the default control framework for the robot -->
+    <!-- <xacro:include filename="gazebo_control.xacro" /> -->
+    <xacro:include filename="ros2_control.xacro" />
 </robot>

File: echo_bot_pkg/description/robot_base.xacro (robot description, xacro)
@@ -73,5 +73,5 @@
         <collision>
             <geometry>
-                <cylinder radius="0.05" length="0.04" />
+                <sphere radius="0.05" />
             </geometry>
         </collision>
@@ -101,5 +101,5 @@
         <collision>
             <geometry>
-                <cylinder radius="0.05" length="0.04" />
+                <sphere radius="0.05" />
             </geometry>
         </collision>
