Commit message: Add SLAM

File: echo_bot_pkg/description/robot_base.xacro (robot description, xacro)
@@ -21,5 +21,5 @@
     </link>
     <!-- BASE FOOTPRINT -->
-    <!-- <joint name="base_footprint_joint" type="fixed">
+    <joint name="base_footprint_joint" type="fixed">
         <parent link="base_link"/>
         <child link="base_footprint"/>
@@ -27,5 +27,5 @@
     </joint>
     <link name="base_footprint">
-    </link> -->
+    </link>
     <!--CHASSIS LINK-->
     <joint name="chassis_joint" type="fixed">
